File: pmod-intermediary.kicad_pcb (KiCad board)
At the start: 2 copper layers, 46 x 16 mm, 15 parts, among them J1 Conn_02x06_male_plug, J2 Conn_02x06_pins, J3 Conn_02x06_female_receptable, J4 Conn_01x03, J5 Conn_01x03, J6 Conn_01x03, J7 Conn_02x02_Odd_Even, J8 Conn_01x03

Commit message: production files, pdf
Parts:
- removed J7: Conn_02x02_Odd_Even, Connector_PinHeader_2.54mm:PinHeader_2x02_P2.54mm_Vertical
Routing:
- net /out_gnd_11: track 41.1 -> 34.9 mm, vias 1 -> 2
- net /out_pwr_6: track 36.3 -> 34.0 mm
- net /out_pwr_12: track 39.3 -> 39.6 mm, vias 1 -> 2
Other:
- board text added: "+"
- board text added: "-"
- board text added: "/\ GND sense R \/ PWR"
- board text added: "GND"
- board text added: "P1"
- board text added: "P10"
- board text added: "P11"
- board text added: "P12"
- board text added: "P2"
- board text added: "P3"
- board text added: "P4"
- board text added: "P5"
- board text added: "P6"
- board text added: "P7"
- board text added: "P8"
- board text added: "P9"
- board text added: "PWR"
- board text added: "on"
- board text added: "on^"
