File: pmod-intermediary.kicad_sch (KiCad schematic)
At the start: 15 parts, among them J1 Conn_02x06_male_plug, J2 Conn_02x06_pins, J3 Conn_02x06_female_receptable, J4 Conn_01x03, J5 Conn_01x03, J6 Conn_01x03, J7 Conn_02x02_Odd_Even, J8 Conn_01x03

Commit message: production files, pdf
Parts:
- removed J7: Conn_02x02_Odd_Even, Connector_PinHeader_2.54mm:PinHeader_2x02_P2.54mm_Vertical, symbol Connector_Generic:Conn_02x02_Odd_Even
Changed lines of the file:
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@@
     (effects (font (size 1.27 1.27)) (justify left bottom))
-  )
-  (label "out_pwr_6" (at 43.18 77.47 180) (fields_autoplaced)
-    (effects (font (size 1.27 1.27)) (justify right bottom))
   )
   (label "out_gnd_5" (at 80.01 41.91 180) (fields_autoplaced)
@@
     (effects (font (size 1.27 1.27)) (justify left bottom))
   )
-  (label "out_gnd_11" (at 55.88 74.93 0) (fields_autoplaced)
-    (effects (font (size 1.27 1.27)) (justify left bottom))
-  )
   (label "out_gnd_11" (at 104.14 58.42 0) (fields_autoplaced)
     (effects (font (size 1.27 1.27)) (justify left bottom))
@@
     (effects (font (size 1.27 1.27)) (justify right bottom))
   )
-  (label "out_gnd_5" (at 55.88 77.47 0) (fields_autoplaced)
-    (effects (font (size 1.27 1.27)) (justify left bottom))
-  )
   (label "in_8" (at 58.42 34.29 0) (fields_autoplaced)
     (effects (font (size 1.27 1.27)) (justify left bottom))
@@
   )
   (label "in_2" (at 80.01 34.29 180) (fields_autoplaced)
-    (effects (font (size 1.27 1.27)) (justify right bottom))
-  )
-  (label "out_pwr_12" (at 43.18 74.93 180) (fields_autoplaced)
     (effects (font (size 1.27 1.27)) (justify right bottom))
   )
@@
         )
       )
-      (project "pmod-measuring-adapter"
+      (project "pmod-intermediary"
         (path "/fa61056b-7d43-4fdf-a61b-eec01ae57378"
           (reference "D1") (unit 1)
@@
     (pin "2")
     (instances
-      (project "pmod-measuring-adapter"
+      (project "pmod-intermediary"
         (path "/fa61056b-7d43-4fdf-a61b-eec01ae57378"
           (reference "R3") (unit 1)
@@
     (pin "2")
     (instances
-      (project "pmod-measuring-adapter"
+      (project "pmod-intermediary"
         (path "/fa61056b-7d43-4fdf-a61b-eec01ae57378"
           (reference "R2") (unit 1)
@@
     (pin "3")
     (instances
-      (project "pmod-measuring-adapter"
+      (project "pmod-intermediary"
         (path "/fa61056b-7d43-4fdf-a61b-eec01ae57378"
           (reference "J6") (unit 1)
@@
     )
   )
-  (symbol (lib_id "Connector_Generic:Conn_02x02_Odd_Even") (at 48.26 74.93 0) (unit 1)
-    (in_bom yes) (on_board yes) (dnp no) (fields_autoplaced)
-    (property "Reference" "J7" (at 49.53 69.85 0)
-      (effects (font (size 1.27 1.27)))
-    )
-    (property "Value" "Conn_02x02_Odd_Even" (at 49.53 72.39 0)
-      (effects (font (size 1.27 1.27)))
-    )
-    (property "Footprint" "Connector_PinHeader_2.54mm:PinHeader_2x02_P2.54mm_Vertical" (at 48.26 74.93 0)
-      (effects (font (size 1.27 1.27)) hide)
-    )
-    (property "Datasheet" "~" (at 48.26 74.93 0)
-      (effects (font (size 1.27 1.27)) hide)
-    )
-    (pin "1")
-    (pin "2")
-    (pin "3")
-    (pin "4")
-    (instances
-      (project "pmod-measuring-adapter"
-        (path "/fa61056b-7d43-4fdf-a61b-eec01ae57378"
-          (reference "J7") (unit 1)
-        )
-      )
-    )
-  )
   (symbol (lib_id "Connector_Generic:Conn_01x03") (at 128.27 68.58 180) (unit 1)
     (in_bom yes) (on_board yes) (dnp no) (fields_autoplaced)
@@
     (pin "3")
     (instances
-      (project "pmod-measuring-adapter"
+      (project "pmod-intermediary"
         (path "/fa61056b-7d43-4fdf-a61b-eec01ae57378"
           (reference "J5") (unit 1)
@@
     (pin "2")
     (instances
-      (project "pmod-measuring-adapter"
+      (project "pmod-intermediary"
         (path "/fa61056b-7d43-4fdf-a61b-eec01ae57378"
           (reference "R1") (unit 1)
@@
         )
       )
-      (project "pmod-measuring-adapter"
+      (project "pmod-intermediary"
         (path "/fa61056b-7d43-4fdf-a61b-eec01ae57378"
           (reference "R5") (unit 1)
@@
     (pin "9")
     (instances
-      (project "pmod-measuring-adapter"
+      (project "pmod-intermediary"
         (path "/fa61056b-7d43-4fdf-a61b-eec01ae57378"
           (reference "J3") (unit 1)
@@
         )
       )
-      (project "pmod-measuring-adapter"
+      (project "pmod-intermediary"
         (path "/fa61056b-7d43-4fdf-a61b-eec01ae57378"
           (reference "C1") (unit 1)
@@
     (pin "3")
     (instances
-      (project "pmod-measuring-adapter"
+      (project "pmod-intermediary"
         (path "/fa61056b-7d43-4fdf-a61b-eec01ae57378"
           (reference "J8") (unit 1)
@@
     (pin "9")
     (instances
-      (project "pmod-measuring-adapter"
+      (project "pmod-intermediary"
         (path "/fa61056b-7d43-4fdf-a61b-eec01ae57378"
           (reference "J2") (unit 1)
@@
     (pin "2")
     (instances
-      (project "pmod-measuring-adapter"
+      (project "pmod-intermediary"
         (path "/fa61056b-7d43-4fdf-a61b-eec01ae57378"
           (reference "R4") (unit 1)
@@
     (pin "9")
     (instances
-      (project "pmod-measuring-adapter"
+      (project "pmod-intermediary"
         (path "/fa61056b-7d43-4fdf-a61b-eec01ae57378"
           (reference "J1") (unit 1)
@@
     (pin "3")
     (instances
-      (project "pmod-measuring-adapter"
+      (project "pmod-intermediary"
         (path "/fa61056b-7d43-4fdf-a61b-eec01ae57378"
           (reference "J4") (unit 1)
